File: incandescentDriver.brd (EAGLE design)
At the start: 100.3 x 47.2 mm, 36 parts, among them IC2 788TV, IC5 74LS595N, J1 HEADER, J10 HEADER, J11 POWER_JACKPTH_LOCK, J2 HEADER, J3 HEADER, J4 HEADER, J5 HEADER, J6 HEADER, J7 HEADER, J8 HEADER, J9 HEADER

Commit message: working on BOM
Parts:
- C1: value 1uF -> 0.1uF
- IC2: value 788TV -> 7805
- R1: value M10LOCK -> 10K
- R2: value M10LOCK -> 1K
Changed lines of the file:
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@@
 </autorouter>
 <elements>
-<element name="J1" library="Livestream" package="1X02-5.08-SCREWTERM" value="HEADER" x="5.62" y="42.18"/>
-<element name="J2" library="Livestream" package="1X02-5.08-SCREWTERM" value="HEADER" x="18.32" y="42.18"/>
-<element name="J3" library="Livestream" package="1X02-5.08-SCREWTERM" value="HEADER" x="31.02" y="42.18"/>
-<element name="J4" library="Livestream" package="1X02-5.08-SCREWTERM" value="HEADER" x="43.72" y="42.18"/>
+<element name="J1" library="Livestream" package="1X02-5.08-SCREWTERM" value="HEADER" x="5.62" y="42.18">
+<attribute name="PARTNO" value="OSTTC022162" x="5.62" y="42.18" size="1.778" layer="27" display="off"/>
+</element>
+<element name="J2" library="Livestream" package="1X02-5.08-SCREWTERM" value="HEADER" x="18.32" y="42.18">
+<attribute name="PARTNO" value="OSTTC022162" x="18.32" y="42.18" size="1.778" layer="27" display="off"/>
+</element>
+<element name="J3" library="Livestream" package="1X02-5.08-SCREWTERM" value="HEADER" x="31.02" y="42.18">
+<attribute name="PARTNO" value="OSTTC022162" x="31.02" y="42.18" size="1.778" layer="27" display="off"/>
+</element>
+<element name="J4" library="Livestream" package="1X02-5.08-SCREWTERM" value="HEADER" x="43.72" y="42.18">
+<attribute name="PARTNO" value="OSTTC022162" x="43.72" y="42.18" size="1.778" layer="27" display="off"/>
+</element>
 <element name="IC5" library="SparkFun-DigitalIC" package="DIL16" value="74LS595N" x="41.45" y="14.2">
-<attribute name="PARTNO" value="74VHC595MTCX" x="65.58" y="-40.41" size="1.778" layer="27" display="off"/>
+<attribute name="PARTNO" value="SN74HC164N" x="65.58" y="-40.41" size="1.778" layer="27" display="off"/>
 </element>
-<element name="C1" library="SparkFun-Capacitors" package="CAP-PTH-SMALL" value="1uF" x="21.14" y="18.08" rot="R180">
-<attribute name="PARTNO" value="CL21B105KOFNNNE" x="-10.61" y="104.44" size="1.778" layer="27" rot="R180" display="off"/>
+<element name="C1" library="SparkFun-Capacitors" package="CAP-PTH-SMALL" value="0.1uF" x="21.14" y="18.08" rot="R180">
+<attribute name="PARTNO" value="SR295E104MAR" x="-10.61" y="104.44" size="1.778" layer="27" rot="R180" display="off"/>
 </element>
-<element name="JP3" library="SparkFun-Connectors" package="1X05_LOCK" value="" x="5.62" y="23.13" rot="R270"/>
-<element name="JP1" library="SparkFun-Connectors" package="1X05_LOCK" value="" x="94.52" y="14.24" rot="R90"/>
-<element name="J11" library="SparkFun-Connectors" package="POWER_JACK_PTH_LOCK" value="POWER_JACKPTH_LOCK" x="68.98" y="7.09" rot="R270"/>
+<element name="JP3" library="SparkFun-Connectors" package="1X05_LOCK" value="" x="5.62" y="23.13" rot="R270">
+<attribute name="PARTNO" value="M20-9960545" x="5.62" y="23.13" size="1.778" layer="27" rot="R270" display="off"/>
+</element>
+<element name="JP1" library="SparkFun-Connectors" package="1X05_LOCK" value="" x="94.52" y="14.24" rot="R90">
+<attribute name="PARTNO" value="M20-9960545" x="94.52" y="14.24" size="1.778" layer="27" rot="R90" display="off"/>
+</element>
+<element name="J11" library="SparkFun-Connectors" package="POWER_JACK_PTH_LOCK" value="POWER_JACKPTH_LOCK" x="68.98" y="7.09" rot="R270">
+<attribute name="PARTNO" value="PJ-202A" x="68.98" y="7.09" size="1.778" layer="27" rot="R270" display="off"/>
+</element>
 <element name="J9" library="Livestream" package="1X02-5.08-SCREWTERM" value="HEADER" x="86.9" y="6.62" rot="R90">
 <attribute name="DNP" value="T" x="164.37" y="25.67" size="1.778" layer="27" rot="R90" display="off"/>
+<attribute name="PARTNO" value="OSTTC022162" x="86.9" y="6.62" size="1.778" layer="27" rot="R90" display="off"/>
 </element>
 <element name="J10" library="Livestream" package="1X02-5.08-SCREWTERM" value="HEADER" x="96.56" y="6.62" rot="R90">
 <attribute name="DNP" value="T" x="174.03" y="37.1" size="1.778" layer="27" rot="R90" display="off"/>
+<attribute name="PARTNO" value="OSTTC022162" x="96.56" y="6.62" size="1.778" layer="27" rot="R90" display="off"/>
 </element>
-<element name="R1" library="SparkFun-Connectors" package="1X10_LOCK" value="M10LOCK" x="24.94" y="5.04"/>
-<element name="Q2" library="transistor-power" package="TO220BV" value="" x="18.32" y="37.1"/>
-<element name="Q1" library="transistor-power" package="TO220BV" value="" x="5.62" y="37.1"/>
-<element name="Q4" library="transistor-power" package="TO220BV" value="" x="43.72" y="37.1"/>
-<element name="Q3" library="transistor-power" package="TO220BV" value="" x="31.02" y="37.1"/>
-<element name="J5" library="Livestream" package="1X02-5.08-SCREWTERM" value="HEADER" x="56.42" y="42.18"/>
-<element name="J6" library="Livestream" package="1X02-5.08-SCREWTERM" value="HEADER" x="69.12" y="42.18"/>
-<element name="J7" library="Livestream" package="1X02-5.08-SCREWTERM" value="HEADER" x="81.82" y="42.18"/>
-<element name="J8" library="Livestream" package="1X02-5.08-SCREWTERM" value="HEADER" x="94.52" y="42.18"/>
-<element name="Q6" library="transistor-power" package="TO220BV" value="" x="69.12" y="37.1"/>
-<element name="Q5" library="transistor-power" package="TO220BV" value="" x="56.42" y="37.1"/>
-<element name="Q8" library="transistor-power" package="TO220BV" value="" x="94.52" y="37.1"/>
-<element name="Q7" library="transistor-power" package="TO220BV" value="" x="81.82" y="37.1"/>
-<element name="R2" library="SparkFun-Connectors" package="1X10_LOCK" value="M10LOCK" x="29.75" y="23.13"/>
+<element name="R1" library="SparkFun-Connectors" package="1X10_LOCK" value="10K" x="24.94" y="5.04">
+<attribute name="PARTNO" value="L101S103LF" x="24.94" y="5.04" size="1.778" layer="27" display="off"/>
+</element>
+<element name="Q2" library="transistor-power" package="TO220BV" value="" x="18.32" y="37.1">
+<attribute name="PARTNO" value="FQP13N10L" x="18.32" y="37.1" size="1.778" layer="27" display="off"/>
+</element>
+<element name="Q1" library="transistor-power" package="TO220BV" value="" x="5.62" y="37.1">
+<attribute name="PARTNO" value="FQP13N10L" x="5.62" y="37.1" size="1.778" layer="27" display="off"/>
+</element>
+<element name="Q4" library="transistor-power" package="TO220BV" value="" x="43.72" y="37.1">
+<attribute name="PARTNO" value="FQP13N10L" x="43.72" y="37.1" size="1.778" layer="27" display="off"/>
+</element>
+<element name="Q3" library="transistor-power" package="TO220BV" value="" x="31.02" y="37.1">
+<attribute name="PARTNO" value="FQP13N10L" x="31.02" y="37.1" size="1.778" layer="27" display="off"/>
+</element>
+<element name="J5" library="Livestream" package="1X02-5.08-SCREWTERM" value="HEADER" x="56.42" y="42.18">
+<attribute name="PARTNO" value="OSTTC022162" x="56.42" y="42.18" size="1.778" layer="27" display="off"/>
+</element>
+<element name="J6" library="Livestream" package="1X02-5.08-SCREWTERM" value="HEADER" x="69.12" y="42.18">
+<attribute name="PARTNO" value="OSTTC022162" x="69.12" y="42.18" size="1.778" layer="27" display="off"/>
+</element>
+<element name="J7" library="Livestream" package="1X02-5.08-SCREWTERM" value="HEADER" x="81.82" y="42.18">
+<attribute name="PARTNO" value="OSTTC022162" x="81.82" y="42.18" size="1.778" layer="27" display="off"/>
+</element>
+<element name="J8" library="Livestream" package="1X02-5.08-SCREWTERM" value="HEADER" x="94.52" y="42.18">
+<attribute name="PARTNO" value="OSTTC022162" x="94.52" y="42.18" size="1.778" layer="27" display="off"/>
+</element>
+<element name="Q6" library="transistor-power" package="TO220BV" value="" x="69.12" y="37.1">
+<attribute name="PARTNO" value="FQP13N10L" x="69.12" y="37.1" size="1.778" layer="27" display="off"/>
+</element>
+<element name="Q5" library="transistor-power" package="TO220BV" value="" x="56.42" y="37.1">
+<attribute name="PARTNO" value="FQP13N10L" x="56.42" y="37.1" size="1.778" layer="27" display="off"/>
+</element>
+<element name="Q8" library="transistor-power" package="TO220BV" value="" x="94.52" y="37.1">
+<attribute name="PARTNO" value="FQP13N10L" x="94.52" y="37.1" size="1.778" layer="27" display="off"/>
+</element>
+<element name="Q7" library="transistor-power" package="TO220BV" value="" x="81.82" y="37.1">
+<attribute name="PARTNO" value="FQP13N10L" x="81.82" y="37.1" size="1.778" layer="27" display="off"/>
+</element>
+<element name="R2" library="SparkFun-Connectors" package="1X10_LOCK" value="1K" x="29.75" y="23.13">
+<attribute name="PARTNO" value="4609X-101-102LF" x="29.75" y="23.13" size="1.778" layer="27" display="off"/>
+</element>
 <element name="LED1" library="adafruit" package="LED5MM" value="" x="5.62" y="29.48" rot="R90"/>
 <element name="LED2" library="adafruit" package="LED5MM" value="" x="18.32" y="29.48" rot="R90"/>
@@
 <element name="LED7" library="adafruit" package="LED5MM" value="" x="81.82" y="29.48" rot="R90"/>
 <element name="LED8" library="adafruit" package="LED5MM" value="" x="94.52" y="29.48" rot="R90"/>
-<element name="C2" library="SparkFun-Capacitors" package="CAP-PTH-SMALL" value="0.33uF" x="75.74" y="19.67" rot="R180"/>
-<element name="C3" library="SparkFun-Capacitors" package="CAP-PTH-SMALL" value="0.1uF" x="66.84" y="15.52" rot="R270"/>
-<element name="IC2" library="linear" package="TO220V" value="788TV" x="74.1" y="11.94" rot="R180"/>
+<element name="C2" library="SparkFun-Capacitors" package="CAP-PTH-SMALL" value="0.33uF" x="75.74" y="19.67" rot="R180">
+<attribute name="PARTNO" value="FK24X7R1H334K" x="75.74" y="19.67" size="1.778" layer="27" rot="R180" display="off"/>
+</element>
+<element name="C3" library="SparkFun-Capacitors" package="CAP-PTH-SMALL" value="0.1uF" x="66.84" y="15.52" rot="R270">
+<attribute name="PARTNO" value="SR295E104MAR" x="66.84" y="15.52" size="1.778" layer="27" rot="R270" display="off"/>
+</element>
+<element name="IC2" library="linear" package="TO220V" value="7805" x="74.1" y="11.94" rot="R180">
+<attribute name="PARTNO" value="NCP7805TG" x="74.1" y="11.94" size="1.778" layer="27" rot="R180" display="off"/>
+</element>
 </elements>
 <signals>
