File: incandescentDriver.sch (EAGLE design)
At the start: 36 parts, among them IC2 788TV, IC5 74LS595N, J1 HEADER, J10 HEADER, J11 POWER_JACKPTH_LOCK, J2 HEADER, J3 HEADER, J4 HEADER, J5 HEADER, J6 HEADER, J7 HEADER, J8 HEADER, J9 HEADER

Commit message: working on BOM
Parts:
- C1: value 1uF -> 0.1uF; PARTNO CL21B105KOFNNNE -> SR295E104MAR
- C2: PARTNO (none) -> FK24X7R1H334K
- C3: PARTNO (none) -> SR295E104MAR
- IC2: value 788TV -> 7805; PARTNO (none) -> NCP7805TG
- IC5: PARTNO 74VHC595MTCX -> SN74HC164N
- J1, J10, J2, J3, J4, J5, J6, J7, J8, J9: PARTNO (none) -> OSTTC022162
- J11: PARTNO (none) -> PJ-202A
- JP1, JP3: PARTNO (none) -> M20-9960545
- Q1, Q2, Q3, Q4, Q5, Q6, Q7, Q8: PARTNO (none) -> FQP13N10L
- R1: value M10LOCK -> 10K; PARTNO (none) -> L101S103LF
- R2: value M10LOCK -> 1K; PARTNO (none) -> 4609X-101-102LF
